File: Keyboard/EagleSchematics/keyboard Right.sch (EAGLE design)
At the start: 73 parts

Commit message: Cleaned up my keyboard schematics.
Parts:
- removed D30: 1N4004, diode:1N4004
- added FN_LED1: TLLG4400, led:TLLG4400
- added R10, R11, R2, R3, R4, R5, R6, R7, R8, R9: 10K, resistor:R-US_0204/7
- renumbered LED1 to CP_LED1, MINUX to MINUS
Connections:
- removed net N$44: CP_LED1.C, U$27.GND
- removed net N$45: D30.A, FN.PIN-2
- removed net N$46: BACKSPACE.PIN-1
- removed net N$50: ].PIN-1
- removed net N$53: BACKSLASH.PIN-1
- removed net N$56: ENTER.PIN-1
- removed net N$59: SHIFT.PIN-1
- removed net N$6: D31.C, U$27.6/PWM
- new net N$25: FN_LED1.A, R2.2
- new net N$57: R2.1, U$27.6/PWM
- net N$13: now also BACKSLASH.PIN-1, ].PIN-1
- net N$14: now also ENTER.PIN-1
- net N$2: now also SHIFT.PIN-1
- net N$21: now also FN.PIN-2, R3.2, U$27.7/RX3; no longer FN.PIN-1
- net N$31: now also R6.2, U$27.10/TX2/PWM; no longer U$27.8/TX3
- net N$35: now also CP_LED1.C, FN.PIN-1, FN_LED1.C, R10.1, R11.1, R3.1, R4.1, R5.1, R6.1, R7.1, R8.1, R9.1, U$27.GND; no longer D30.C
- net N$36: now also R7.2, U$27.11/MOSI; no longer U$27.9/RX2/PWM
- net N$4: now also BACKSPACE.PIN-1
- net N$41: now also D4.C, R8.2, U$27.12/MISO; no longer U$27.10/TX2/PWM
- net N$48: now also R5.2, U$27.9/RX2/PWM; no longer U$27.7/RX3
- net N$49: now also R9.2, U$27.13/SCK/LED; no longer U$27.11/MOSI
- net N$55: now also D31.C, R4.2, U$27.8/TX3
- net N$62: now also R11.2, U$27.15/A1/T; no longer U$27.13/SCK/LED
- net OPTION: now also R10.2, U$27.14/A0; no longer U$27.12/MISO
