File: Keyboard/EagleSchematics/keyboard left.sch (EAGLE design)
At the start: 63 parts

Commit message: Cleaned up my keyboard schematics.
Parts:
- removed D30: 1N4004, diode:1N4004
- added FN_LED1: TLLG4400, led:TLLG4400
- added R10, R2, R3, R4, R5, R6, R7, R8, R9: 10K, resistor:R-US_0204/7
- renumbered LED1 to CP_LED1
Connections:
- removed net N$44: CP_LED1.C, U$27.GND
- removed net N$45: D30.A, SPACE.PIN-2
- new net N$48: D7.C, R4.2, U$27.8/TX3
- new net N$49: D10.C, D16.C, D22.C, D28.C, D3.C, R8.2, U$27.12/MISO
- new net N$57: R2.1, U$27.6/PWM
- new net N$62: D1.C, D14.C, D20.C, D8.C, R10.2, U$27.14/A0
- new net OPTION: D15.C, D2.C, D21.C, D27.C, D9.C, R9.2, U$27.13/SCK/LED
- net N$1: no longer FN.PIN-1, SPACE.PIN-1
- net N$21: now also FN.PIN-2, R3.2, U$27.7/RX3; no longer D15.C, D2.C, D21.C, D27.C, D9.C, U$27.11/MOSI
- net N$24: now also SPACE.PIN-2; no longer FN.PIN-2
- net N$25: now also FN_LED1.A, R2.2; no longer D10.C, D16.C, D22.C, D28.C, D3.C, U$27.10/TX2/PWM
- net N$31: now also D13.C, D19.C, D25.C, D6.C, R5.2; no longer D11.C, D17.C, D23.C, D29.C
- net N$35: now also CP_LED1.C, FN.PIN-1, FN_LED1.C, R10.1, R3.1, R4.1, R5.1, R6.1, R7.1, R8.1, R9.1, U$27.GND; no longer D12.C, D18.C, D24.C, D30.C, D5.C, U$27.8/TX3
- net N$36: now also D12.C, D18.C, D24.C, D26.C, D5.C, R6.2, U$27.10/TX2/PWM; no longer D13.C, D19.C, D25.C, D6.C, U$27.7/RX3
- net N$41: now also D11.C, D17.C, D23.C, D29.C, D4.C, R7.2, U$27.11/MOSI; no longer D7.C, U$27.6/PWM
- net N$6: now also SPACE.PIN-1; no longer D1.C, D14.C, D20.C, D26.C, D8.C, U$27.12/MISO
Other:
- moved on the sheet: D26
